File: diy-schematics.kicad_pcb (KiCad board)
At the start: 2 copper layers, 22 parts, among them J1 MICCON, J2 GAINCON, J3 AudioJack2, J4 USB_C_Receptacle_USB2.0, U1 THAT1512PO8-U1, U2 NMA0515SC

Commit message: FG update
Connections:
- J3 pad S: Earth -> Net-(J3-PadS)
- J4 pad S1: Net-(C4-Pad2) -> Net-(J4-PadS1)

Commit message: misc changes
Connections:
- J3 pad S: Net-(J3-PadS) -> Earth
- J4 pad S1: Net-(J4-PadS1) -> Net-(C4-Pad2)
