File: diy-schematics.sch (KiCad schematic (older format))
At the start: 22 parts, among them J1 MICCON, J2 GAINCON, J3 AudioJack2, J4 USB_C_Receptacle_USB2.0, U1 NMA0515SC, U1 THAT1512PO8-U

Commit message: pcb layout
Parts:
- C1, C2, C4, C5, C6, C7: footprint (none) -> Capacitor_SMD:C_0805_2012Metric
- C8: renamed from C2; footprint (none) -> Capacitor_SMD:C_0805_2012Metric
- J1, J2: footprint (none) -> Connector_JST:JST_XH_B2B-XH-A_1x02_P2.50mm_Vertical
- J3: footprint (none) -> Connector_Audio:Jack_3.5mm_QingPu_WQP-PJ398SM_Vertical_CircularHoles
- J4: footprint (none) -> Connector_USB:USB_C_Receptacle_Palconn_UTC16-G
- N-JFET1: renamed from N-JFET; footprint (none) -> Package_TO_SOT_THT:TO-72-4
- R1, R2, R3, R4, R5, R6, R7, R8: footprint (none) -> Resistor_SMD:R_0603_1608Metric
- U1: value THAT1512PO8-U -> THAT1512PO8-U1; footprint that-corp-DIL08 -> Package_DIP:DIP-8_W7.62mm_Socket
- renumbered U1 to U2
Changed lines of the file:
@@
 F 0 "R2" H 2520 4996 50  0000 L CNN
 F 1 "2.2kΩ" H 2520 4905 50  0000 L CNN
-F 2 "" V 2380 4950 50  0001 C CNN
+F 2 "Resistor_SMD:R_0603_1608Metric" V 2380 4950 50  0001 C CNN
 F 3 "~" H 2450 4950 50  0001 C CNN
 	1    2450 4950
@@
 F 0 "C1" V 3552 3950 50  0000 C CNN
 F 1 "22uF" V 3461 3950 50  0000 C CNN
-F 2 "" H 3338 3800 50  0001 C CNN
+F 2 "Capacitor_SMD:C_0805_2012Metric" H 3338 3800 50  0001 C CNN
 F 3 "~" H 3300 3950 50  0001 C CNN
 	1    3300 3950
@@
 F 0 "C2" V 3552 4550 50  0000 C CNN
 F 1 "22uF" V 3461 4550 50  0000 C CNN
-F 2 "" H 3338 4400 50  0001 C CNN
+F 2 "Capacitor_SMD:C_0805_2012Metric" H 3338 4400 50  0001 C CNN
 F 3 "~" H 3300 4550 50  0001 C CNN
 	1    3300 4550
@@
 F 0 "R3" H 4120 3646 50  0000 L CNN
 F 1 "3.9kΩ" H 4120 3555 50  0000 L CNN
-F 2 "" V 3980 3600 50  0001 C CNN
+F 2 "Resistor_SMD:R_0603_1608Metric" V 3980 3600 50  0001 C CNN
 F 3 "~" H 4050 3600 50  0001 C CNN
 	1    4050 3600
@@
 F 0 "R4" H 4120 4996 50  0000 L CNN
 F 1 "3.9kΩ" H 4120 4905 50  0000 L CNN
-F 2 "" V 3980 4950 50  0001 C CNN
+F 2 "Resistor_SMD:R_0603_1608Metric" V 3980 4950 50  0001 C CNN
 F 3 "~" H 4050 4950 50  0001 C CNN
 	1    4050 4950
@@
 $EndComp
 $Comp
-L Device:C C2
+L Device:C C8
 U 1 1 61C27CF6
 P 6400 4100
-F 0 "C2" V 6652 4100 50  0000 C CNN
+F 0 "C8" V 6652 4100 50  0000 C CNN
 F 1 "22uF" V 6561 4100 50  0000 C CNN
-F 2 "" H 6438 3950 50  0001 C CNN
+F 2 "Capacitor_SMD:C_0805_2012Metric" H 6438 3950 50  0001 C CNN
 F 3 "~" H 6400 4100 50  0001 C CNN
 	1    6400 4100
@@
 F 0 "C7" H 6118 5746 50  0000 L CNN
 F 1 "2200uF 16V" H 6118 5655 50  0000 L CNN
-F 2 "" H 6038 5550 50  0001 C CNN
+F 2 "Capacitor_SMD:C_0805_2012Metric" H 6038 5550 50  0001 C CNN
 F 3 "~" H 6000 5700 50  0001 C CNN
 	1    6000 5700
@@
 F 0 "C6" H 6118 2596 50  0000 L CNN
 F 1 "2200uF 16V" H 6118 2505 50  0000 L CNN
-F 2 "" H 6038 2400 50  0001 C CNN
+F 2 "Capacitor_SMD:C_0805_2012Metric" H 6038 2400 50  0001 C CNN
 F 3 "~" H 6000 2550 50  0001 C CNN
 	1    6000 2550
@@
 F 0 "R5" H 5620 2596 50  0000 L CNN
 F 1 "2.2kΩ" H 5620 2505 50  0000 L CNN
-F 2 "" V 5480 2550 50  0001 C CNN
+F 2 "Resistor_SMD:R_0603_1608Metric" V 5480 2550 50  0001 C CNN
 F 3 "~" H 5550 2550 50  0001 C CNN
 	1    5550 2550
@@
 F 0 "R6" H 5620 5746 50  0000 L CNN
 F 1 "2.2kΩ" H 5620 5655 50  0000 L CNN
-F 2 "" V 5480 5700 50  0001 C CNN
+F 2 "Resistor_SMD:R_0603_1608Metric" V 5480 5700 50  0001 C CNN
 F 3 "~" H 5550 5700 50  0001 C CNN
 	1    5550 5700
@@
 F 0 "R7" V 7107 2400 50  0000 C CNN
 F 1 "100Ω" V 7016 2400 50  0000 C CNN
-F 2 "" V 6830 2400 50  0001 C CNN
+F 2 "Resistor_SMD:R_0603_1608Metric" V 6830 2400 50  0001 C CNN
 F 3 "~" H 6900 2400 50  0001 C CNN
 	1    6900 2400
@@
 $EndComp
 $Comp
-L Regulator_Switching:NMA0515SC U1
+L Regulator_Switching:NMA0515SC U2
 U 1 1 61C2AA61
 P 7850 4000
-F 0 "U1" H 7850 3533 50  0000 C CNN
+F 0 "U2" H 7850 3533 50  0000 C CNN
 F 1 "NMA0515SC" H 7850 3624 50  0000 C CNN
 F 2 "Converter_DCDC:Converter_DCDC_muRata_NMAxxxxSC_THT" H 7850 3650 50  0001 C CIN
@@
 F 0 "C4" H 8618 4096 50  0000 L CNN
 F 1 "2200uF" H 8618 4005 50  0000 L CNN
-F 2 "" H 8538 3900 50  0001 C CNN
+F 2 "Capacitor_SMD:C_0805_2012Metric" H 8538 3900 50  0001 C CNN
 F 3 "~" H 8500 4050 50  0001 C CNN
 	1    8500 4050
@@
 F 0 "C5" H 9168 4096 50  0000 L CNN
 F 1 "2200uF" H 9168 4005 50  0000 L CNN
-F 2 "" H 9088 3900 50  0001 C CNN
+F 2 "Capacitor_SMD:C_0805_2012Metric" H 9088 3900 50  0001 C CNN
 F 3 "~" H 9050 4050 50  0001 C CNN
 	1    9050 4050
@@
 U 1 1 61C4FA52
 P 5050 4250
-F 0 "U1" H 5894 4296 50  0000 L CNN
-F 1 "THAT1512PO8-U" H 5894 4205 50  0000 L CNN
-F 2 "that-corp-DIL08" H 5050 4400 50  0001 C CNN
+F 0 "U1" H 4950 4350 50  0000 L CNN
+F 1 "THAT1512PO8-U1" H 4700 4250 50  0000 L CNN
+F 2 "Package_DIP:DIP-8_W7.62mm_Socket" H 5050 4400 50  0001 C CNN
 F 3 "" H 5050 4250 50  0001 C CNN
 	1    5050 4250
@@
 $EndComp
 $Comp
-L power:Earth #PWR?
+L power:Earth #PWR0101
 U 1 1 61C51431
 P 5250 4850
-F 0 "#PWR?" H 5250 4600 50  0001 C CNN
+F 0 "#PWR0101" H 5250 4600 50  0001 C CNN
 F 1 "Earth" H 5250 4700 50  0001 C CNN
 F 2 "" H 5250 4850 50  0001 C CNN
@@
 $EndComp
 $Comp
-L power:Earth #PWR?
+L power:Earth #PWR0102
 U 1 1 61C52553
 P 5550 5500
-F 0 "#PWR?" H 5550 5250 50  0001 C CNN
+F 0 "#PWR0102" H 5550 5250 50  0001 C CNN
 F 1 "Earth" H 5550 5350 50  0001 C CNN
 F 2 "" H 5550 5500 50  0001 C CNN
@@
 $EndComp
 $Comp
-L power:Earth #PWR?
+L power:Earth #PWR0103
 U 1 1 61C52AF8
 P 6000 5500
-F 0 "#PWR?" H 6000 5250 50  0001 C CNN
+F 0 "#PWR0103" H 6000 5250 50  0001 C CNN
 F 1 "Earth" H 6000 5350 50  0001 C CNN
 F 2 "" H 6000 5500 50  0001 C CNN
@@
 $EndComp
 $Comp
-L power:Earth #PWR?
+L power:Earth #PWR0104
 U 1 1 61C52F85
 P 5550 2750
-F 0 "#PWR?" H 5550 2500 50  0001 C CNN
+F 0 "#PWR0104" H 5550 2500 50  0001 C CNN
 F 1 "Earth" H 5550 2600 50  0001 C CNN
 F 2 "" H 5550 2750 50  0001 C CNN
@@
 $EndComp
 $Comp
-L power:Earth #PWR?
+L power:Earth #PWR0105
 U 1 1 61C532AB
 P 6000 2750
-F 0 "#PWR?" H 6000 2500 50  0001 C CNN
+F 0 "#PWR0105" H 6000 2500 50  0001 C CNN
 F 1 "Earth" H 6000 2600 50  0001 C CNN
 F 2 "" H 6000 2750 50  0001 C CNN
@@
 $EndComp
 $Comp
-L power:Earth #PWR?
+L power:Earth #PWR0106
 U 1 1 61C53513
 P 1250 4350
-F 0 "#PWR?" H 1250 4100 50  0001 C CNN
+F 0 "#PWR0106" H 1250 4100 50  0001 C CNN
 F 1 "Earth" H 1250 4200 50  0001 C CNN
 F 2 "" H 1250 4350 50  0001 C CNN
@@
 $EndComp
 $Comp
-L power:Earth #PWR?
+L power:Earth #PWR0107
 U 1 1 61C53DD7
 P 7350 4000
-F 0 "#PWR?" H 7350 3750 50  0001 C CNN
+F 0 "#PWR0107" H 7350 3750 50  0001 C CNN
 F 1 "Earth" H 7350 3850 50  0001 C CNN
 F 2 "" H 7350 4000 50  0001 C CNN
@@
 $EndComp
 $Comp
-L power:Earth #PWR?
+L power:Earth #PWR0108
 U 1 1 61C55B83
 P 4050 3350
-F 0 "#PWR?" H 4050 3100 50  0001 C CNN
+F 0 "#PWR0108" H 4050 3100 50  0001 C CNN
 F 1 "Earth" H 4050 3200 50  0001 C CNN
 F 2 "" H 4050 3350 50  0001 C CNN
@@
 $EndComp
 $Comp
-L power:Earth #PWR?
+L power:Earth #PWR0109
 U 1 1 61C56138
 P 4050 5250
-F 0 "#PWR?" H 4050 5000 50  0001 C CNN
+F 0 "#PWR0109" H 4050 5000 50  0001 C CNN
 F 1 "Earth" H 4050 5100 50  0001 C CNN
 F 2 "" H 4050 5250 50  0001 C CNN
@@
 F 0 "R1" H 2380 3554 50  0000 R CNN
 F 1 "2.2kΩ" H 2380 3645 50  0000 R CNN
-F 2 "" V 2380 3600 50  0001 C CNN
+F 2 "Resistor_SMD:R_0603_1608Metric" V 2380 3600 50  0001 C CNN
 F 3 "~" H 2450 3600 50  0001 C CNN
 	1    2450 3600
@@
 	1950 4450 1950 4550
 $Comp
-L Device:Q_NJFET_SGD N-JFET
+L Device:Q_NJFET_SGD N-JFET1
 U 1 1 61C25741
 P 1850 4250
-F 0 "N-JFET" H 2040 4296 50  0000 L CNN
+F 0 "N-JFET1" H 2040 4296 50  0000 L CNN
 F 1 "2N4416" H 2040 4205 50  0000 L CNN
-F 2 "" H 2050 4350 50  0001 C CNN
+F 2 "Package_TO_SOT_THT:TO-72-4" H 2050 4350 50  0001 C CNN
 F 3 "~" H 1850 4250 50  0001 C CNN
 	1    1850 4250
@@
 F 0 "J1" H 842 4025 50  0000 C CNN
 F 1 "MICCON" H 842 4116 50  0000 C CNN
-F 2 "" H 950 4350 50  0001 C CNN
+F 2 "Connector_JST:JST_XH_B2B-XH-A_1x02_P2.50mm_Vertical" H 950 4350 50  0001 C CNN
 F 3 "~" H 950 4350 50  0001 C CNN
 	1    950  4350
@@
 F 0 "J2" H 4400 4200 50  0000 C CNN
 F 1 "GAINCON" H 4450 4300 50  0000 C CNN
-F 2 "" H 4250 4300 50  0001 C CNN
+F 2 "Connector_JST:JST_XH_B2B-XH-A_1x02_P2.50mm_Vertical" H 4250 4300 50  0001 C CNN
 F 3 "~" H 4250 4300 50  0001 C CNN
 	1    4250 4300
@@
 F 0 "J3" H 6570 4083 50  0000 R CNN
 F 1 "AudioJack2" H 6570 4174 50  0000 R CNN
-F 2 "" H 6750 4100 50  0001 C CNN
+F 2 "Connector_Audio:Jack_3.5mm_QingPu_WQP-PJ398SM_Vertical_CircularHoles" H 6750 4100 50  0001 C CNN
 F 3 "~" H 6750 4100 50  0001 C CNN
 	1    6750 4100
@@
 F 0 "R8" H 6970 5896 50  0000 L CNN
 F 1 "100Ω" H 6970 5805 50  0000 L CNN
-F 2 "" V 6830 5850 50  0001 C CNN
+F 2 "Resistor_SMD:R_0603_1608Metric" V 6830 5850 50  0001 C CNN
 F 3 "~" H 6900 5850 50  0001 C CNN
 	1    6900 5850
@@
 F 0 "J4" H 9770 3797 50  0000 R CNN
 F 1 "USB_C_Receptacle_USB2.0" H 10600 4700 50  0000 R CNN
-F 2 "" H 10350 3950 50  0001 C CNN
+F 2 "Connector_USB:USB_C_Receptacle_Palconn_UTC16-G" H 10350 3950 50  0001 C CNN
 F 3 "https://www.usb.org/sites/default/files/documents/usb_type-c.zip" H 10350 3950 50  0001 C CNN
 	1    10200 3950

Commit message: misc changes
Parts:
- added C10, C8, C9: 100nF, symbol Device:C
- R2, R3, R4, R5, R6, R7, R8: footprint Resistor_SMD:R_0603_1608Metric -> Resistor_THT:R_Axial_DIN0207_L6.3mm_D2.5mm_P10.16mm_Horizontal
- U1: symbol that-corp:THAT1512PO8-U -> diy-schematics-rescue:THAT1512PO8-U-that-corp
Connections:
- net Earth: now also J3.S, C10.1, C9.2
- net at C6.1, R1.2, R5.1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: now also C9.1
- net at C7.2, R2.2, R6.2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: now also C10.2
- net at C4.1, C5.1, J4.A4 (VBUS)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: now also C8.1
- net at C4.2, C5.2, J4.A1 (GND)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: now also J4.S1 (SHIELD), C8.2
- no-connect marks 0 -> 8
Changed lines of the file:
@@
 F 0 "R2" H 2520 4996 50  0000 L CNN
 F 1 "2.2kΩ" H 2520 4905 50  0000 L CNN
-F 2 "Resistor_SMD:R_0603_1608Metric" V 2380 4950 50  0001 C CNN
+F 2 "Resistor_THT:R_Axial_DIN0207_L6.3mm_D2.5mm_P10.16mm_Horizontal" V 2380 4950 50  0001 C CNN
 F 3 "~" H 2450 4950 50  0001 C CNN
 	1    2450 4950
@@
 F 0 "R3" H 4120 3646 50  0000 L CNN
 F 1 "3.9kΩ" H 4120 3555 50  0000 L CNN
-F 2 "Resistor_SMD:R_0603_1608Metric" V 3980 3600 50  0001 C CNN
+F 2 "Resistor_THT:R_Axial_DIN0207_L6.3mm_D2.5mm_P10.16mm_Horizontal" V 3980 3600 50  0001 C CNN
 F 3 "~" H 4050 3600 50  0001 C CNN
 	1    4050 3600
@@
 F 0 "R4" H 4120 4996 50  0000 L CNN
 F 1 "3.9kΩ" H 4120 4905 50  0000 L CNN
-F 2 "Resistor_SMD:R_0603_1608Metric" V 3980 4950 50  0001 C CNN
+F 2 "Resistor_THT:R_Axial_DIN0207_L6.3mm_D2.5mm_P10.16mm_Horizontal" V 3980 4950 50  0001 C CNN
 F 3 "~" H 4050 4950 50  0001 C CNN
 	1    4050 4950
@@
 F 0 "R5" H 5620 2596 50  0000 L CNN
 F 1 "2.2kΩ" H 5620 2505 50  0000 L CNN
-F 2 "Resistor_SMD:R_0603_1608Metric" V 5480 2550 50  0001 C CNN
+F 2 "Resistor_THT:R_Axial_DIN0207_L6.3mm_D2.5mm_P10.16mm_Horizontal" V 5480 2550 50  0001 C CNN
 F 3 "~" H 5550 2550 50  0001 C CNN
 	1    5550 2550
@@
 F 0 "R6" H 5620 5746 50  0000 L CNN
 F 1 "2.2kΩ" H 5620 5655 50  0000 L CNN
-F 2 "Resistor_SMD:R_0603_1608Metric" V 5480 5700 50  0001 C CNN
+F 2 "Resistor_THT:R_Axial_DIN0207_L6.3mm_D2.5mm_P10.16mm_Horizontal" V 5480 5700 50  0001 C CNN
 F 3 "~" H 5550 5700 50  0001 C CNN
 	1    5550 5700
@@
 F 0 "R7" V 7107 2400 50  0000 C CNN
 F 1 "100Ω" V 7016 2400 50  0000 C CNN
-F 2 "Resistor_SMD:R_0603_1608Metric" V 6830 2400 50  0001 C CNN
+F 2 "Resistor_THT:R_Axial_DIN0207_L6.3mm_D2.5mm_P10.16mm_Horizontal" V 6830 2400 50  0001 C CNN
 F 3 "~" H 6900 2400 50  0001 C CNN
 	1    6900 2400
@@
 $EndComp
 $Comp
-L that-corp:THAT1512PO8-U U1
+L diy-schematics-rescue:THAT1512PO8-U-that-corp U1
 U 1 1 61C4FA52
 P 5050 4250
@@
 Connection ~ 5050 2400
 Wire Wire Line
-	5050 2400 5550 2400
+	5050 2400 5250 2400
 Wire Wire Line
 	6000 5850 5550 5850
@@
 F 0 "R8" H 6970 5896 50  0000 L CNN
 F 1 "100Ω" H 6970 5805 50  0000 L CNN
-F 2 "Resistor_SMD:R_0603_1608Metric" V 6830 5850 50  0001 C CNN
+F 2 "Resistor_THT:R_Axial_DIN0207_L6.3mm_D2.5mm_P10.16mm_Horizontal" V 6830 5850 50  0001 C CNN
 F 3 "~" H 6900 5850 50  0001 C CNN
 	1    6900 5850
@@
 	9050 4200 9050 5100
 Wire Wire Line
-	9050 5100 10200 5100
+	9050 5100 9900 5100
 Wire Wire Line
 	10800 3050 10800 3350
@@
 Connection ~ 5050 5850
 Wire Wire Line
-	5050 5850 5550 5850
+	5050 5850 5250 5850
 Wire Wire Line
 	1950 4550 2450 4550
@@
 Connection ~ 8500 3800
 Wire Wire Line
-	8500 3800 9050 3800
+	8500 3800 8800 3800
 Wire Wire Line
 	8350 4200 8500 4200
 Wire Wire Line
-	8500 4200 9050 4200
+	8500 4200 8800 4200
 Connection ~ 8500 4200
 Connection ~ 9050 4200
+$Comp
+L power:Earth #PWR0110
+U 1 1 61D1B253
+P 6550 4300
+F 0 "#PWR0110" H 6550 4050 50  0001 C CNN
+F 1 "Earth" H 6550 4150 50  0001 C CNN
+F 2 "" H 6550 4300 50  0001 C CNN
+F 3 "~" H 6550 4300 50  0001 C CNN
+	1    6550 4300
+	1    0    0    -1
+$EndComp
+Wire Wire Line
+	6550 4200 6550 4300
+Wire Wire Line
+	9900 4850 9900 5100
+Connection ~ 9900 5100
+Wire Wire Line
+	9900 5100 10200 5100
+NoConn ~ 10850 3550
+NoConn ~ 10800 3550
+NoConn ~ 10800 3650
+NoConn ~ 10800 3850
+NoConn ~ 10800 3950
+NoConn ~ 10800 4050
+NoConn ~ 10800 4150
+NoConn ~ 10800 4450
+$Comp
+L Device:C C8
+U 1 1 61D6146E
+P 8800 4050
+F 0 "C8" H 8915 4096 50  0000 L CNN
+F 1 "100nF" H 8915 4005 50  0000 L CNN
+F 2 "" H 8838 3900 50  0001 C CNN
+F 3 "~" H 8800 4050 50  0001 C CNN
+	1    8800 4050
+	1    0    0    -1
+$EndComp
+Connection ~ 8800 4200
+Wire Wire Line
+	8800 4200 9050 4200
+Wire Wire Line
+	8800 3900 8800 3800
+Connection ~ 8800 3800
+Wire Wire Line
+	8800 3800 9050 3800
+$Comp
+L Device:C C10
+U 1 1 61D63F44
+P 5250 5700
+F 0 "C10" H 5365 5746 50  0000 L CNN
+F 1 "100nF" H 5365 5655 50  0000 L CNN
+F 2 "" H 5288 5550 50  0001 C CNN
+F 3 "~" H 5250 5700 50  0001 C CNN
+	1    5250 5700
+	1    0    0    -1
+$EndComp
+Connection ~ 5250 5850
+Wire Wire Line
+	5250 5850 5550 5850
+$Comp
+L Device:C C9
+U 1 1 61D7A27B
+P 5250 2550
+F 0 "C9" H 5365 2596 50  0000 L CNN
+F 1 "100nF" H 5365 2505 50  0000 L CNN
+F 2 "" H 5288 2400 50  0001 C CNN
+F 3 "~" H 5250 2550 50  0001 C CNN
+	1    5250 2550
+	1    0    0    -1
+$EndComp
+Connection ~ 5250 2400
+Wire Wire Line
+	5250 2400 5550 2400
+$Comp
+L power:Earth #PWR?
+U 1 1 61D7D39D
+P 5250 2750
+F 0 "#PWR?" H 5250 2500 50  0001 C CNN
+F 1 "Earth" H 5250 2600 50  0001 C CNN
+F 2 "" H 5250 2750 50  0001 C CNN
+F 3 "~" H 5250 2750 50  0001 C CNN
+	1    5250 2750
+	1    0    0    -1
+$EndComp
+$Comp
+L power:Earth #PWR?
+U 1 1 61D7DBE2
+P 5250 5500
+F 0 "#PWR?" H 5250 5250 50  0001 C CNN
+F 1 "Earth" H 5250 5350 50  0001 C CNN
+F 2 "" H 5250 5500 50  0001 C CNN
+F 3 "~" H 5250 5500 50  0001 C CNN
+	1    5250 5500
+	-1   0    0    1
+$EndComp
+Wire Wire Line
+	5250 2700 5250 2750
+Wire Wire Line
+	5250 5550 5250 5500
 $EndSCHEMATC

Commit message: FG update
Parts:
- removed C8: 100nF, symbol Device:C
- removed J3: AudioJack2, Connector_Audio:Jack_3.5mm_QingPu_WQP-PJ398SM_Vertical_CircularHoles, symbol Connector:AudioJack2
- removed J4: USB_C_Receptacle_USB2.0, Connector_USB:USB_C_Receptacle_Palconn_UTC16-G, symbol Connector:USB_C_Receptacle_USB2.0
- added C3: 100n, Capacitor_THT:C_Rect_L7.0mm_W2.5mm_P5.00mm, symbol Device:C
- added J3: AudioJack2_Ground, symbol Connector:AudioJack2_Ground
- added J4: USB_B_Micro, symbol Connector:USB_B_Micro
- added J6: MIC_CON1, symbol Connector_Generic:Conn_01x03
- added J7: MIC_CON2, symbol Connector_Generic:Conn_01x03
- added J?: Conn_01x04, symbol Connector_Generic:Conn_01x04
- C10, C9: value 100nF -> 100n; footprint (none) -> Capacitor_THT:C_Rect_L7.0mm_W2.5mm_P5.00mm
- J1: value MICCON -> CAPSULE
- R2, R3, R4, R5, R6, R7, R8: footprint Resistor_THT:R_Axial_DIN0207_L6.3mm_D2.5mm_P10.16mm_Horizontal -> Resistor_SMD:R_0603_1608Metric
Connections:
- net Earth: now also C10.2, C4.2, C5.2, R3.2, R6.2, U2.2 (VIN-), C3.2, J3.G, J4.5 (GND), J4.6 (Shield), J6.2 (Pin_2), J7.2 (Pin_2), J?.4 (Pin_4); no longer C10.1, R3.1, R6.1
- net at C1.1, R1.1: now also J6.1 (Pin_1); no longer N-JFET1.3 (D)
- net at C6.1, R1.2, R5.1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: now also C3.1; no longer C9.1
- net at C2.1, R2.1: now also J6.3 (Pin_3); no longer N-JFET1.1 (S)
- net at C7.2, R2.2, R8.1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: now also C9.1, R6.1; no longer C10.2, R6.2
- net at C1.2, U1.2 (IN-): now also R3.1; no longer R3.2
- net at C8.2: now also J3.S, J3.T
- net +15V: now reaches R7.2, U2.6 (VOUT+)
- net -15V: now reaches R8.2, U2.4 (VOUT-)
- net VBUS: now reaches C4.1, C5.1, U2.1 (VIN+)
- net VBUS: now also C10.1, J4.1 (VBUS), J?.1 (Pin_1)
- new net: J7.3 (Pin_3), N-JFET1.1 (S)
- new net: J7.1 (Pin_1), N-JFET1.3 (D)
- new net: J4.2 (D-), J?.3 (Pin_3)
- new net: J4.3 (D+), J?.2 (Pin_2)
- no-connect marks 8 -> 0
Other:
- note added: "Microphone capsule connected via cable"
- moved on the sheet: C4, C7, J1, N-JFET1, R3, R4, R6
